File: led.sch (EAGLE design)
At the start: 3 parts

Commit message: Whoops! Forgot a resistor!
Parts:
- added R1: 220, SparkFun-Resistors:RESISTORAXIAL-0.3
Connections:
- new net N$2: D1.A, R1.1
- net VCC: now also R1.2; no longer D1.A
Changed lines of the file:
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@@
 <part name="S1" library="SparkFun-Switches" deviceset="SWITCH-SPDT" device="-PTH-11.6X4.0MM-LOCK"/>
 <part name="J1" library="SparkFun-Connectors" deviceset="CONN_02" device="LOCK"/>
+<part name="R1" library="SparkFun-Resistors" deviceset="RESISTOR" device="AXIAL-0.3" value="220"/>
 </parts>
 <sheets>
@@
 <attribute name="VALUE" x="22.86" y="68.326" size="1.778" layer="96" font="vector" rot="R180"/>
 <attribute name="NAME" x="22.86" y="57.912" size="1.778" layer="95" font="vector" rot="R180"/>
+</instance>
+<instance part="R1" gate="G$1" x="-15.24" y="73.66" smashed="yes" rot="R90">
+<attribute name="NAME" x="-16.764" y="73.66" size="1.778" layer="95" font="vector" rot="R90" align="bottom-center"/>
+<attribute name="VALUE" x="-13.716" y="73.66" size="1.778" layer="96" font="vector" rot="R90" align="top-center"/>
 </instance>
 </instances>
@@
 <net name="VCC" class="0">
 <segment>
-<pinref part="D1" gate="D1" pin="A"/>
 <pinref part="SUPPLY1" gate="G$1" pin="VCC"/>
-<wire x1="-15.24" y1="68.58" x2="-15.24" y2="78.74" width="0.1524" layer="91"/>
 <wire x1="-15.24" y1="78.74" x2="7.62" y2="78.74" width="0.1524" layer="91"/>
 <wire x1="7.62" y1="78.74" x2="7.62" y2="63.5" width="0.1524" layer="91"/>
 <pinref part="J1" gate="G$1" pin="1"/>
 <wire x1="7.62" y1="63.5" x2="12.7" y2="63.5" width="0.1524" layer="91"/>
+<pinref part="R1" gate="G$1" pin="2"/>
 <junction x="-15.24" y="78.74"/>
 </segment>
 </net>
+<net name="N$2" class="0">
+<segment>
+<pinref part="D1" gate="D1" pin="A"/>
+<pinref part="R1" gate="G$1" pin="1"/>
+</segment>
+</net>
